Commit message: Add files via upload

File: autonoship_simulation/urdf/container_ship.xacro (robot description, xacro)
@@ -1,22 +1,22 @@
 <?xml version="1.0"?>
 <robot name="container_ship" xmlns:xacro="http://ros.org/wiki/xacro">
-    <xacro:arg name="windType" default="global" />
-    <xacro:arg name="waterType" default="global" />
-    <xacro:property name="windType" value="$(arg windType)" />
-    <xacro:property name="waterType" value="$(arg waterType)" />
-    <xacro:property name="dampingXYZ" value="1.88 10 6.66" />
-    <xacro:property name="angularDampingXYZ" value="2 15 2" />
-    <xacro:property name="PI" value="3.1415926535897931"/>
-    <!-- Body properties -->
-    <xacro:property name="front_body_mass" value="0.5"/>
-    <xacro:property name="back_body_mass" value="2"/>
-    <xacro:property name="middle_body_mass" value="143620"/>
-    <xacro:property name="back_water_displaced_mass" value="10"/>
-    <xacro:property name="middle_water_displaced_mass" value="10"/>
-    <xacro:property name="front_water_displaced_mass" value="5"/>
-    <xacro:property name="extraPayload" value="0"/>
-    <xacro:property name="scale" value="1.5"/>
-    <xacro:property name="bl1" value=".1" />
-    <xacro:property name="bl2" value=".1" />
+  <xacro:arg name="windType" default="global" />
+  <xacro:arg name="waterType" default="global" />
+  <xacro:property name="windType" value="$(arg windType)" />
+  <xacro:property name="waterType" value="$(arg waterType)" />
+  <xacro:property name="dampingXYZ" value="1.88 10 6.66" />
+  <xacro:property name="angularDampingXYZ" value="2 15 2" />
+  <xacro:property name="PI" value="3.1415926535897931"/>
+  <!-- Body properties -->
+  <xacro:property name="front_body_mass" value="0.5"/>
+  <xacro:property name="back_body_mass" value="2"/>
+  <xacro:property name="middle_body_mass" value="143620"/>
+  <xacro:property name="back_water_displaced_mass" value="10"/>
+  <xacro:property name="middle_water_displaced_mass" value="10"/>
+  <xacro:property name="front_water_displaced_mass" value="5"/>
+  <xacro:property name="extraPayload" value="0"/>
+  <xacro:property name="scale" value="1.5"/>
+  <xacro:property name="bl1" value=".1" />
+  <xacro:property name="bl2" value=".1" />
     <link name="base_footprint">
       <visual>
@@ -26,4 +26,5 @@
         </geometry>
       </visual>
+      <!--
       <collision>
         <origin rpy="0 0 0" xyz="0 0 0"/>
@@ -31,5 +32,11 @@
            <box size="0.001 0.001 0.001" />
         </geometry>
+        <surface>
+          <contact>
+            <collide_bitmask>0x01</collide_bitmask>
+          </contact>
+        </surface>
       </collision>
+      -->
       <inertial>
         <origin rpy="0 0 0" xyz="0 0 0"/>
@@ -49,12 +56,21 @@
           </geometry>
         </visual>
+        <!--
         <collision>
           <origin rpy="0 0 0" xyz="105.2 21.54 -10"/>
           <geometry>
-             <box size="334 43.08 15" />  <!--  334 174 30  -->
+             <box size="334 43.08 15" />          -->
+             <!--  334 174 30  -->
              <!-- <box size="311.6 62.622 40" /> -->
              <!-- <mesh filename="package://autonoship_simulation/rudder_ship/Ship_construture_process.dae" scale="${scale} ${scale} ${scale}"/> -->
+          <!--
           </geometry>
+          <surface>
+            <contact>
+              <collide_bitmask>0x01</collide_bitmask>
+            </contact>
+          </surface>
         </collision>
+        -->
         <inertial>
           <!-- <origin rpy="0 0 0" xyz="-155.8 -31.311 -10"/> -->
@@ -81,9 +97,16 @@
         <inertia ixx="0.000140625" ixy="0.0" ixz="0.0" iyy="0.000140625" iyz="0.0" izz="0.00028125"/>
       </inertial>
+      <!--
       <collision>
         <geometry>
           <cylinder radius="0.075" length="0.15"/>
         </geometry>
+        <surface>
+          <contact>
+            <collide_bitmask>0x01</collide_bitmask>
+          </contact>
+        </surface>
       </collision>
+      -->
       <visual>
         <geometry>
@@ -104,9 +127,16 @@
         <inertia ixx="0.0001667" ixy="0.0" ixz="0.0" iyy="0.0001667" iyz="0.0" izz="0.0001667"/>
       </inertial>
+      <!--
       <collision>
         <geometry>
           <box size="0.15 1 0.1" />
         </geometry>
+        <surface>
+          <contact>
+            <collide_bitmask>0x01</collide_bitmask>
+          </contact>
+        </surface>
       </collision>
+      -->
       <visual>
         <geometry>

File: autonoship_simulation/urdf/container_ship_noradar.xacro (robot description, xacro)
@@ -1,22 +1,22 @@
 <?xml version="1.0"?>
 <robot name="container_ship" xmlns:xacro="http://ros.org/wiki/xacro">
-    <xacro:arg name="windType" default="global" />
-    <xacro:arg name="waterType" default="global" />
-    <xacro:property name="windType" value="$(arg windType)" />
-    <xacro:property name="waterType" value="$(arg waterType)" />
-    <xacro:property name="dampingXYZ" value="1.88 10 6.66" />
-    <xacro:property name="angularDampingXYZ" value="2 15 2" />
-    <xacro:property name="PI" value="3.1415926535897931"/>
-    <!-- Body properties -->
-    <xacro:property name="front_body_mass" value="0.5"/>
-    <xacro:property name="back_body_mass" value="2"/>
-    <xacro:property name="middle_body_mass" value="200000"/>
-    <xacro:property name="back_water_displaced_mass" value="10"/>
-    <xacro:property name="middle_water_displaced_mass" value="10"/>
-    <xacro:property name="front_water_displaced_mass" value="5"/>
-    <xacro:property name="extraPayload" value="0"/>
-    <xacro:property name="scale" value="1.5"/>
-    <xacro:property name="bl1" value=".1" />
-    <xacro:property name="bl2" value=".1" />
+  <xacro:arg name="windType" default="global" />
+  <xacro:arg name="waterType" default="global" />
+  <xacro:property name="windType" value="$(arg windType)" />
+  <xacro:property name="waterType" value="$(arg waterType)" />
+  <xacro:property name="dampingXYZ" value="1.88 10 6.66" />
+  <xacro:property name="angularDampingXYZ" value="2 15 2" />
+  <xacro:property name="PI" value="3.1415926535897931"/>
+  <!-- Body properties -->
+  <xacro:property name="front_body_mass" value="0.5"/>
+  <xacro:property name="back_body_mass" value="2"/>
+  <xacro:property name="middle_body_mass" value="200000"/>
+  <xacro:property name="back_water_displaced_mass" value="10"/>
+  <xacro:property name="middle_water_displaced_mass" value="10"/>
+  <xacro:property name="front_water_displaced_mass" value="5"/>
+  <xacro:property name="extraPayload" value="0"/>
+  <xacro:property name="scale" value="1.5"/>
+  <xacro:property name="bl1" value=".1" />
+  <xacro:property name="bl2" value=".1" />
     <link name="base_footprint">
       <visual>
@@ -31,4 +31,9 @@
            <box size="0.001 0.001 0.001" />
         </geometry>
+        <surface>
+          <contact>
+            <collide_bitmask>0x02</collide_bitmask>
+          </contact>
+        </surface>
       </collision>
       <inertial>
@@ -56,4 +61,9 @@
              <!-- <mesh filename="package://autonoship_simulation/rudder_ship/Ship_construture_process.dae" scale="${scale} ${scale} ${scale}"/> -->
           </geometry>
+          <surface>
+            <contact>
+              <collide_bitmask>0x02</collide_bitmask>
+            </contact>
+          </surface>
         </collision>
         <inertial>
